File: PCB Shield.kicad_sch (KiCad schematic)
At the start: 47 parts, among them J1 Conn_01x20, J10 TB002-500-02BE, J12 TB002-500-02BE, J13 TB002-500-02BE, J14 TB002-500-02BE, J15 TB002-500-02BE, J16 TB002-500-02BE, J17 TB002-500-02BE, J18 TB002-500-02BE, J2 Conn_01x08_Socket, J3 Conn_01x20, J4 Conn_01x20, J5 Conn_01x20, J6 Conn_01x04_Socket, J7 Conn_01x04_Socket, J8 Conn_01x04_Socket, J9 OSTT7020150, Q1 IRLML2502TRPBF, SW1 C1353VQNAA, U2 74AHCT125S14-13, U3 ESDA6V1L

Commit message: all shematic changes made
Parts:
- removed J8: Conn_01x04_Socket, Connector_PinSocket_2.54mm:PinSocket_1x04_P2.54mm_Vertical, symbol Connector:Conn_01x04_Socket
- added R2, R3: 4k7, 196_Project_Footprints:RC1206FR-074K7L, symbol 196_Project:RC1206FR-074K7L
Connections:
- net +5V: now also J6.3 (Pin_3), J7.3 (Pin_3), R2.2, R3.2; no longer J6.1 (Pin_1), J7.1 (Pin_1)
- net SCL / IO9: now also J6.2 (Pin_2), J7.2 (Pin_2), R3.1; no longer J6.3 (Pin_3), J7.3 (Pin_3)
- net SDA / IO8: now also J6.1 (Pin_1), J7.1 (Pin_1), R2.1; no longer J6.2 (Pin_2), J7.2 (Pin_2)
Other:
- note added: "Logic shifter not necessary for short wires, but I want to allow room wide connections. Aka, if I need a longer connection from this circuit to an LED wall, then I want that option."
- note added: "Pull up resistors"
- note added: "Two I2C outputs"
- note removed: "Not necessary for short wires, but I want to allow room wide connections. Aka, if I need a longer connection from this circuit to an LED wall, then I want that option."
- moved on the sheet: J10, J15, J6, R6, R7, R8, R9
