File: PCB Shield.kicad_sch (KiCad schematic)
At the start: 53 parts, among them J1 Conn_1to20, J10 TB002-500-02BE, J11 TB002-500-02BE, J12 TB002-500-02BE, J13 TB002-500-02BE, J14 TB002-500-02BE, J15 TB002-500-02BE, J16 TB002-500-02BE, J2 Conn_01x08_Socket, J3 Conn_1to20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

Commit message: quick
Parts:
- C1, C7: symbol 196_Project:1206B104K500BD -> 196_Project:CL31B104KBCNNNC
- C2: symbol 196_Project:1206B105K250JC -> 196_Project:CL31B105KAHNNNE
- Q1: symbol 196_Project:IRLML2502TRPBF -> 196_Project:DMN2075U-7
Changed lines of the file:
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@@
 	)
 	(junction
-		(at 135.89 87.63)
-		(diameter 0)
-		(color 0 0 0 0)
-	)
-	(junction
 		(at 214.63 62.23)
 		(diameter 0)
@@
 	)
 	(junction
-		(at 161.29 72.39)
-		(diameter 0)
-		(color 0 0 0 0)
-	)
-	(junction
 		(at 139.7 26.67)
 		(diameter 0)
@@
 	(wire
 		(pts
-			(xy 135.89 86.36) (xy 135.89 87.63)
-		)
-		(stroke
-			(width 0)
-			(type default)
-		)
-	)
-	(wire
-		(pts
 			(xy 266.7 109.22) (xy 269.24 109.22)
 		)
@@
 	(wire
 		(pts
-			(xy 160.02 72.39) (xy 161.29 72.39)
-		)
-		(stroke
-			(width 0)
-			(type default)
-		)
-	)
-	(wire
-		(pts
 			(xy 273.05 62.23) (xy 273.05 64.77)
 		)
@@
 	)
 	(symbol
-		(lib_id "196_Project:1206B104K500BD")
+		(lib_id "196_Project:CL31B104KBCNNNC")
 		(at 267.97 88.9 270)
 		(unit 1)
@@
 			)
 		)
-		(property "Datasheet" "https://mm.digikey.com/Volume0/opasdata/d220001/medias/docus/6490/3372_1206B104K500BD.pdf"
+		(property "Datasheet" ""
 			(at 267.97 88.9 0)
 			(hide yes)
@@
 	)
 	(symbol
-		(lib_id "196_Project:IRLML2502TRPBF")
+		(lib_id "196_Project:DMN2075U-7")
 		(at 26.67 121.92 0)
 		(unit 1)
@@
 			)
 		)
-		(property "Datasheet" "https://www.infineon.com/assets/row/public/documents/24/49/infineon-irlml2502-datasheet-en.pdf"
+		(property "Datasheet" ""
 			(at 24.638 108.966 0)
 			(hide yes)
@@
 	)
 	(symbol
-		(lib_id "196_Project:1206B105K250JC")
+		(lib_id "196_Project:CL31B105KAHNNNE")
 		(at 143.51 87.63 180)
 		(unit 1)
@@
 			)
 		)
-		(property "Datasheet" "https://mm.digikey.com/Volume0/opasdata/d220001/medias/docus/5660/3372_1206B105K250JC.pdf"
+		(property "Datasheet" ""
 			(at 145.288 100.33 0)
 			(hide yes)
@@
 			)
 		)
-		(property "Description" "CAP CER 1UF 25V X7R 1206"
+		(property "Description" "CAP CER 0.1UF 50V X7R 1206"
 			(at 145.288 100.33 0)
 			(hide yes)
@@
 	)
 	(symbol
-		(lib_id "196_Project:1206B104K500BD")
+		(lib_id "196_Project:CL31B104KBCNNNC")
 		(at 135.89 83.82 180)
 		(unit 1)
@@
 			)
 		)
-		(property "Datasheet" "https://mm.digikey.com/Volume0/opasdata/d220001/medias/docus/6490/3372_1206B104K500BD.pdf"
+		(property "Datasheet" ""
 			(at 135.89 83.82 0)
 			(hide yes)

Commit message: finally done ????
Parts:
- C1, C7: footprint 196_Project_Footprints:1206B104K500BD -> 196_Project_Footprints:CL31B104KBCNNNC
- C2: footprint 196_Project_Footprints:1206B105K250JC -> 196_Project_Footprints:CL31B105KAHNNNE
Changed lines of the file:
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@@
 			)
 		)
-		(property "Footprint" "196_Project_Footprints:1206B104K500BD"
+		(property "Footprint" "196_Project_Footprints:CL31B104KBCNNNC"
 			(at 278.638 91.186 0)
 			(hide yes)
@@
 			)
 		)
-		(property "Description" "CONN HEADER VERT 20POS 2.54MM"
+		(property "Description" "Generic connector, single row, 01x20, script generated (kicad-library-utils/schlib/autogen/connector/)"
 			(at 115.57 49.53 0)
 			(hide yes)
@@
 			)
 		)
-		(property "Description" "CONN HEADER VERT 20POS 2.54MM"
+		(property "Description" "Generic connector, single row, 01x20, script generated (kicad-library-utils/schlib/autogen/connector/)"
 			(at 131.318 22.86 0)
 			(hide yes)
@@
 			)
 		)
-		(property "Description" "CONN HEADER VERT 8POS 2.54MM"
+		(property "Description" "Generic connector, single row, 01x08, script generated"
 			(at 106.68 116.84 0)
 			(hide yes)
@@
 			)
 		)
-		(property "Description" "CONN HEADER VERT 4POS 2.54MM"
+		(property "Description" "Generic connector, single row, 01x04, script generated"
 			(at 180.34 129.54 0)
 			(hide yes)
@@
 			)
 		)
-		(property "Description" "CONN HEADER VERT 4POS 2.54MM"
+		(property "Description" "Generic connector, single row, 01x04, script generated"
 			(at 152.4 129.54 0)
 			(hide yes)
@@
 			)
 		)
-		(property "Description" "CONN HEADER VERT 20POS 2.54MM"
+		(property "Description" "Generic connector, single row, 01x20, script generated (kicad-library-utils/schlib/autogen/connector/)"
 			(at 122.428 22.86 0)
 			(hide yes)
@@
 			)
 		)
-		(property "Footprint" "196_Project_Footprints:1206B105K250JC"
+		(property "Footprint" "196_Project_Footprints:CL31B105KAHNNNE"
 			(at 141.224 98.298 0)
 			(hide yes)
@@
 			)
 		)
-		(property "Description" "CONN HEADER VERT 20POS 2.54MM"
+		(property "Description" "Generic connector, single row, 01x20, script generated (kicad-library-utils/schlib/autogen/connector/)"
 			(at 106.68 49.53 0)
 			(hide yes)
@@
 			)
 		)
-		(property "Footprint" "196_Project_Footprints:1206B104K500BD"
+		(property "Footprint" "196_Project_Footprints:CL31B104KBCNNNC"
 			(at 133.604 94.488 0)
 			(hide yes)

Commit message: changed switch
Parts:
- J1, J3, J4, J5: MANUFACTURER Würth Elektronik -> Adam Tech; Part Number 61302011121 -> PH1-20-UA
- J2: MANUFACTURER Würth Elektronik -> Adam Tech; Part Number 61300811121 -> PH1-20-UA
- J6, J7: MANUFACTURER Würth Elektronik -> Adam Tech; Part Number 61300411121 -> PH1-20-UA
- SW1: value C1353VQNAA -> GRB066L02BBGGL1; symbol 196_Project:C1353VQNAA -> 196_Project:GRB066L02BBGGL1; MANUFACTURER Bulgin -> CW Industries; Part Number C1353VQNAA -> GRB066L02BBGGL1
Connections:
- net GND: now also SW1.3

Commit message: finished finally and totally. parts ready to order too.
Parts:
- SW1: footprint 196_Project_Footprints:C1353VQNAA -> 196_Project_Footprints:GRB066L02BBGGL1
Changed lines of the file:
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@@
 	(text "Power Supply"
 		(exclude_from_sim no)
-		(at 158.75 60.706 0)
+		(at 157.988 56.642 0)
 		(effects
 			(font
@@
 		(dnp no)
 		(fields_autoplaced yes)
-		(property "Reference" "#PWR022"
+		(property "Reference" "#PWR22"
 			(at 173.99 82.55 0)
 			(hide yes)
@@
 			(project "PCB Shield"
 				(path "/9e193586-b0fa-43d6-aa55-137433de4788"
-					(reference "#PWR022")
+					(reference "#PWR22")
 					(unit 1)
 				)
@@
 			)
 		)
-		(property "Footprint" "196_Project_Footprints:C1353VQNAA"
+		(property "Footprint" "196_Project_Footprints:GRB066L02BBGGL1"
 			(at 163.068 61.722 0)
 			(hide yes)

Commit message: saving myself
Parts:
- removed C3, C4, C5, C6, C8, C9: 470uF, 196_Project_Footprints:25ZLH470MEFC10X12, symbol 196_Project:25ZLH470MEFC10X12.5
- removed C7: 0.1uF, 196_Project_Footprints:CL31B104KBCNNNC, symbol 196_Project:CL31B104KBCNNNC
- removed J10, J11, J12, J13, J14, J15, J16, J9: TB002-500-02BE, 196_Project_Footprints:TB002-500-02BE, symbol 196_Project:TB002-500-02BE
- removed R1, R6, R7, R8, R9: 220, 196_Project_Footprints:RMCF1206FT220R, symbol 196_Project:RMCF1206FT220R
- removed R4: 0, Resistor_SMD:R_1206_3216Metric, symbol 196_Project:RCS12060000Z0EA
- removed U2: 74AHCT125S14-13, 196_Project_Footprints:74AHCT125S14-13, symbol 196_Project:74AHCT125S14-13
- added NT1: NetTie_2, NetTie:NetTie-2_SMD_Pad2.0mm, symbol Device:NetTie_2
- added R1: 10k, Resistor_SMD:R_1206_3216Metric, symbol 196_Project:CRCW120610K0FKEA
- added R10: 150, Resistor_SMD:R_1206_3216Metric, symbol 196_Project:WK73R2BTTD151J
- SW1: MANUFACTURER CW Industries -> (none); Part Number GRB066L02BBGGL1 -> (none)
Connections:
- net +5V: now also C1.1, C2.1, R10.2; no longer SW1.1, U1.1
- net +5Vlimited: now also U1.1, NT1.1; no longer C1.1, C2.1
- net GATE / IO45: now also R1.2
- net GND: now also SW1.4, R1.1; no longer SW1.3
- new net: R10.1, SW1.3
- new net: NT1.2, SW1.1
Other:
- added sheet LED_Power (LED_Power.kicad_sch)
- added sheet Logic_shifter (logic_shifter.kicad_sch)
- note added: "6 terminals for power injections each has a large capacitor to smooth fluctuations"
- note added: "Resistors before data output to allow LED drive 20mA per output (GPIO) 20-80mA Logic shifter not necessary for short wires, but I want to allow room wide connections. Aka, if I need a longer connection from this circuit to an LED wall, then I want that option."
- note removed: "20mA per output (GPIO) 20-80mA"
- note removed: "Coonnector Guide 1 - High / + 2 - Low / - / GND"
- note removed: "Logic shifter for LEDs (prevent flickering)"
- note removed: "Logic shifter not necessary for short wires, but I want to allow room wide connections. Aka, if I need a longer connection from this circuit to an LED wall, then I want that option."
- note removed: "Power Injection Connectors (15-60mA per LED)"
- note removed: "Resistors before data output to allow LED drive"
- moved on the sheet: H1, H2, H3, H4, J8

Commit message: edited and ready
Parts:
- R1: MANUFACTURER (none) -> Vishay Dale; Part Number (none) -> CRCW120610K0FKEA
- R10: MANUFACTURER (none) -> Vishay Dale; Part Number (none) -> RCS1206150RJNEA
- SW1: MANUFACTURER (none) -> CW Industries; Part Number (none) -> GRB066L02BBGGL1
Connections:
- net +5V: now also NT1.2, SW1.1
- net GATE / IO45: now also Q1.1 (G); no longer Q1.2 (G)
- net GND: now also Q1.2 (S); no longer Q1.3 (S)
- net at R2.1: now also Q1.3 (D); no longer Q1.1 (D)
Other:
- moved on the sheet: C1, C2, NT1, U1

Commit message: STILL need to adjust to 30.5mm
Parts:
- LS1: footprint 196_Project_Footprints:AI-3035-TWT-3V-R -> Buzzer_Beeper:Buzzer_12x9.5RM7.6
Connections:
- net GND: now also LS1.2; no longer LS1.N
- net PWM / IO16: now also LS1.1; no longer LS1.P
Other:
- moved on the sheet: C1, C2, H1, H2, H3, H4, J1, J3, J4, J5, J8, NT1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

Commit message: finally order ready
Parts:
- removed H1, H2, H3, H4: MountingHole, 196_Project_Footprints:MountingHole_3.2mm_M3_Pad_Via, symbol Mechanical:MountingHole
- added H1, H2, H3: MountingHole, symbol 196_Project:MountingHole
Connections:
- net GND: now also H1.1, H2.1, H3.1
