File: PCB Shield.kicad_pcb (KiCad board)
At the start: 2 copper layers, 92 x 99 mm, 55 parts, among them J1 Conn_1to20, J10 TB002-500-02BE, J11 TB002-500-02BE, J12 TB002-500-02BE, J13 TB002-500-02BE, J14 TB002-500-02BE, J15 TB002-500-02BE, J16 TB002-500-02BE, J2 Conn_01x08_Socket, J3 Conn_1to20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

Commit message: finally done ????
Parts:
- C1, C7: footprint 196_Project_Footprints:1206B104K500BD -> 196_Project_Footprints:CL31B104KBCNNNC
- C2: footprint 196_Project_Footprints:1206B105K250JC -> 196_Project_Footprints:CL31B105KAHNNNE
- U2: value 74AHCT125S14-13 -> SO14_DIO

Commit message: changed switch
Parts:
- removed SW1: C1353VQNAA, 196_Project_Footprints:C1353VQNAA
- U2: value SO14_DIO -> 74AHCT125S14-13

Commit message: finished finally and totally. parts ready to order too.
Parts:
- added SW1: GRB066L02BBGGL1, 196_Project_Footprints:GRB066L02BBGGL1, F.Cu at (235.9, 75.7)
Routing:
- net +5V: track 208.6 -> 209.3 mm
- net GND: vias 57 -> 55
Changed lines of the file:
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@@
 		)
 	)
+	(footprint "196_Project_Footprints:GRB066L02BBGGL1"
+		(layer "F.Cu")
+		(at 235.8935 75.6985 180)
+		(property "Reference" "SW1"
+			(at 2.032 -0.5 180)
+			(unlocked yes)
+			(layer "F.SilkS")
+			(effects
+				(font
+					(size 1 1)
+					(thickness 0.1)
+				)
+			)
+		)
+		(property "Value" "GRB066L02BBGGL1"
+			(at 0 -7.112 180)
+			(unlocked yes)
+			(layer "F.Fab")
+			(effects
+				(font
+					(size 1 1)
+					(thickness 0.15)
+				)
+			)
+		)
+		(property "Datasheet" ""
+			(at 0 0 180)
+			(unlocked yes)
+			(layer "F.Fab")
+			(hide yes)
+			(effects
+				(font
+					(size 1 1)
+					(thickness 0.15)
+				)
+			)
+		)
+		(property "Description" "SWITCH ROCKER DPST-NO 20A 250V"
+			(at 0 0 180)
+			(unlocked yes)
+			(layer "F.Fab")
+			(hide yes)
+			(effects
+				(font
+					(size 1 1)
+					(thickness 0.15)
+				)
+			)
+		)
+		(property "Part Number" "GRB066L02BBGGL1"
+			(at 0 0 180)
+			(unlocked yes)
+			(layer "F.Fab")
+			(hide yes)
+			(effects
+				(font
+					(size 1 1)
+					(thickness 0.15)
+				)
+			)
+		)
+		(property "Sim.Device" ""
+			(at 0 0 180)
+			(unlocked yes)
+			(layer "F.Fab")
+			(hide yes)
+			(effects
+				(font
+					(size 1 1)
+					(thickness 0.15)
+				)
+			)
+		)
+		(property "Sim.Pins" ""
+			(at 0 0 180)
+			(unlocked yes)
+			(layer "F.Fab")
+			(hide yes)
+			(effects
+				(font
+					(size 1 1)
+					(thickness 0.15)
+				)
+			)
+		)
+		(property "Sim.Type" ""
+			(at 0 0 180)
+			(unlocked yes)
+			(layer "F.Fab")
+			(hide yes)
+			(effects
+				(font
+					(size 1 1)
+					(thickness 0.15)
+				)
+			)
+		)
+		(property "MANUFACTURER" "CW Industries"
+			(at 0 0 180)
+			(unlocked yes)
+			(layer "F.Fab")
+			(hide yes)
+			(effects
+				(font
+					(size 1 1)
+					(thickness 0.15)
+				)
+			)
+		)
+		(sheetname "/")
+		(sheetfile "PCB Shield.kicad_sch")
+		(units
+			(unit
+				(name "A")
+				(pins "1" "2" "3")
+			)
+		)
+		(attr through_hole)
+		(duplicate_pad_numbers_are_jumpers no)
+		(fp_text user "${REFERENCE}"
+			(at 0 -5.612 180)
+			(unlocked yes)
+			(layer "F.Fab")
+			(effects
+				(font
+					(size 1 1)
+					(thickness 0.15)
+				)
+			)
+		)
+		(pad "1" thru_hole circle
+			(at 10.287 1.897 180)
+			(size 3.5 3.5)
+			(drill 2.5)
+			(layers "*.Cu" "*.Mask")
+			(remove_unused_layers no)
+			(net "+5V")
+			(pintype "passive")
+		)
+		(pad "2" thru_hole roundrect
+			(at 6.096 1.77 180)
+			(size 3.5 3.5)
+			(drill 2.5)
+			(layers "*.Cu" "*.Mask")
+			(remove_unused_layers no)
+			(roundrect_rratio 0.07142857143)
+			(net "+5V")
+			(pintype "passive")
+		)
+		(pad "3" thru_hole circle
+			(at 1.778 1.778 180)
+			(size 3.5 3.5)
+			(drill 2.5)
+			(layers "*.Cu" "*.Mask")
+			(remove_unused_layers no)
+			(net "GND")
+			(pintype "passive")
+		)
+		(embedded_fonts no)
+		(model "${KIPRJMOD}/3d models/Round Power Switch.STEP"
+			(offset
+				(xyz 2 -2 0)
+			)
+			(scale
+				(xyz 0.5 0.5 0.5)
+			)
+			(rotate
+				(xyz -90 -0 -0)
+			)
+		)
+	)
 	(footprint "196_Project_Footprints:CMD17-21VGD_TR8"
 		(layer "F.Cu")
@@
 	)
 	(segment
-		(start 220 77)
-		(end 224.425 72.575)
-		(width 3)
-		(layer "F.Cu")
-		(net "+5V")
-	)
-	(segment
-		(start 227.0715 77.147)
-		(end 232.147 77.147)
-		(width 3)
-		(layer "F.Cu")
-		(net "+5V")
-	)
-	(segment
 		(start 241.8375 128.5)
 		(end 241.8375 128.3375)
@@
 	)
 	(segment
+		(start 229.7975 73.9285)
+		(end 229.7975 75.7975)
+		(width 3)
+		(layer "F.Cu")
+		(net "+5V")
+	)
+	(segment
 		(start 241.5 102.5)
 		(end 241.8375 102.5)
@@
 	)
 	(segment
-		(start 227.1985 77.02)
-		(end 227.0715 77.147)
-		(width 3)
-		(layer "F.Cu")
-		(net "+5V")
-	)
-	(segment
 		(start 231 126)
 		(end 229 128)
@@
 	)
 	(segment
-		(start 232.147 77.147)
-		(end 236 81)
-		(width 3)
-		(layer "F.Cu")
-		(net "+5V")
-	)
-	(segment
 		(start 230.83325 139)
 		(end 229 140.83325)
@@
 	)
 	(segment
-		(start 236 81)
-		(end 236 85.0755)
+		(start 236 140)
+		(end 240.3375 140)
 		(width 3)
 		(layer "F.Cu")
@@
 	)
 	(segment
-		(start 236 140)
-		(end 240.3375 140)
+		(start 230.83325 153)
+		(end 229 154.83325)
 		(width 3)
 		(layer "F.Cu")
@@
 	)
 	(segment
-		(start 230.83325 153)
-		(end 229 154.83325)
+		(start 211.0155 73.251601)
+		(end 214.763899 77)
 		(width 3)
 		(layer "F.Cu")
@@
 	)
 	(segment
-		(start 240.3375 154)
-		(end 241.8375 155.5)
+		(start 214.763899 77)
+		(end 222.408 77)
 		(width 3)
 		(layer "F.Cu")
@@
 	)
 	(segment
-		(start 236 127)
-		(end 235 126)
+		(start 240.3375 154)
+		(end 241.8375 155.5)
 		(width 3)
 		(layer "F.Cu")
@@
 	)
 	(segment
-		(start 214.763899 77)
-		(end 220 77)
+		(start 236 127)
+		(end 235 126)
 		(width 3)
 		(layer "F.Cu")
@@
 	)
 	(segment
+		(start 229.74 75.7975)
+		(end 227.0715 78.466)
+		(width 3)
+		(layer "F.Cu")
+		(net "+5V")
+	)
+	(segment
+		(start 236 82)
+		(end 236 85.0755)
+		(width 3)
+		(layer "F.Cu")
+		(net "+5V")
+	)
+	(segment
 		(start 240.3375 114)
 		(end 236 114)
@@
 	)
 	(segment
+		(start 222.408 77)
+		(end 225.6065 73.8015)
+		(width 3)
+		(layer "F.Cu")
+		(net "+5V")
+	)
+	(segment
 		(start 235 153)
 		(end 230.83325 153)
@@
 	)
 	(segment
-		(start 236 140)
-		(end 236 154)
+		(start 229.7975 75.7975)
+		(end 229.74 75.7975)
 		(width 3)
 		(layer "F.Cu")
@@
 	)
 	(segment
-		(start 211.0155 73.251601)
-		(end 214.763899 77)
+		(start 236 140)
+		(end 236 154)
 		(width 3)
 		(layer "F.Cu")
@@
 	)
 	(segment
-		(start 224.425 72.575)
-		(end 227.1985 72.575)
+		(start 229.7975 75.7975)
+		(end 236 82)
 		(width 3)
 		(layer "F.Cu")
@@
 	)
 	(via
-		(at 236 73)
-		(size 1)
-		(drill 0.6)
-		(layers "F.Cu" "B.Cu")
-		(net "GND")
-	)
-	(via
 		(at 219 80)
 		(size 1)
@@
 		(size 1)
 		(drill 0.6)
-		(layers "F.Cu" "B.Cu")
-		(net "GND")
-	)
-	(via
-		(at 231 73)
-		(size 1)
-		(drill 0.6)

Commit message: saved by the bell
Parts:
- added NT1: NetTie_2, NetTie:NetTie-2_SMD_Pad2.0mm, F.Cu at (273.0, 99.0)
- added R1: 10k, Resistor_SMD:R_1206_3216Metric, F.Cu at (272.3, 102.2)
- added R10: 150, Resistor_SMD:R_1206_3216Metric, F.Cu at (272.3, 105.5)
- U2: value 74AHCT125S14-13 -> SO14_DIO
Connections:
- C1 pad 1: +5Vlimited -> +5V
- C2 pad 1: +5Vlimited -> +5V
- Q1 pad 1: Net-(Q1-D) -> GATE / IO45
- Q1 pad 2: GATE / IO45 -> GND
- Q1 pad 3: GND -> Net-(Q1-D)
- SW1 pad 1: +5V -> Net-(NT1-Pad2)
- SW1 pad 3: GND -> Net-(R10-Pad1)
- U1 pad 1: +5V -> +5Vlimited

Commit message: edited and ready
Parts:
- removed the R1 at (214.8, 106.0)
- removed R4: 0, Resistor_SMD:R_1206_3216Metric
- U2: value SO14_DIO -> 74AHCT125S14-13
- moved R1 63.8 mm to (209.0, 110.0)
- moved NT1 49.7 mm to (228.0, 78.0)
- moved R10 47.7 mm to (234.0, 77.0), turned to 180 degrees
- moved C2 19.5 mm to (206.2, 80.0), turned to 180 degrees
- moved C1 19.5 mm to (206.2, 77.0), turned to 180 degrees
- moved U1 12.8 mm to (224.0, 78.0)
- moved R2 5.76 mm to (211.2, 107.0), turned to 180 degrees
- moved SW1 2.92 mm to (238.6, 74.7)
Connections:
- NT1 pad 2: Net-(NT1-Pad2) -> +5V
- SW1 pad 1: Net-(NT1-Pad2) -> +5V
- SW1 pad 4: (no net) -> GND
Routing:
- net +5Vlimited: track 468.9 -> 474.0 mm, vias 6 -> 5
- net Net-(R10-Pad1): track 0.00 -> 4.76 mm
- net Net-(Q1-D): track 5.78 -> 3.04 mm
- net GATE / IO45: track 17.4 -> 14.6 mm
- net +5V: track 209.3 -> 206.9 mm
- net LED split: track 487.7 -> 486.3 mm
- net GND: track 4.59 -> 4.87 mm, vias 55 -> 54
Other:
- board text removed: "switch"

Commit message: STILL need to adjust to 30.5mm
Parts:
- added G***: LOGO, LOGO, F.Cu at (301.0, 39.0)
- added G***: LOGO, LOGO, F.Cu at (166.9, 20.2)
- added G***: LOGO, LOGO, F.Cu at (256.0, 19.6)
- added G***: LOGO, LOGO, F.Cu at (183.0, 88.0)
- added G***: LOGO, LOGO, F.Cu at (133.5, 22.0)
- added G***: LOGO, LOGO, F.Cu at (162.7, -79.7)
- added G***: LOGO, LOGO, F.Cu at (242.0, -90.0)
- added G***: LOGO, LOGO, F.Cu at (198.0, -43.0)
- added G***: LOGO, LOGO, F.Cu at (282.0, -48.0)
- added G***: LOGO, LOGO, F.Cu at (212.1, 24.5)
- added G***: LOGO, LOGO, F.Cu at (238.0, -47.0)
- added G***: LOGO, LOGO, F.Cu at (151.0, -38.1)
- LS1: footprint 196_Project_Footprints:AI-3035-TWT-3V-R -> Buzzer_Beeper:Buzzer_12x9.5RM7.6
- moved LS1 9.18 mm to (191.0, 80.8)
Routing:
- net PWM / IO16: track 39.2 -> 48.4 mm
- net LED split: track 486.3 -> 481.3 mm
Other:
- board text added: "MOVE TO 30.5mm apart"

Commit message: finally order ready
Parts:
- removed G*** (x11): LOGO, LOGO
- removed H4: MountingHole, 196_Project_Footprints:MountingHole_3.2mm_M3_Pad_Via
- moved H3 31.4 mm to (169.3, 139.2)
- moved D8 22.0 mm to (163.0, 92.0), turned to 90 degrees
- moved D7 22.0 mm to (162.0, 70.0), turned to 90 degrees
- moved Q1 6.44 mm to (208.0, 110.0)
- moved R1 4.81 mm to (208.2, 114.8)
- moved R5 4.69 mm to (189.1, 143.3), turned to -90 degrees
- moved ? 2.55 mm to (239.0, 148.5)
- moved D3 2.34 mm to (249.0, 71.2), turned to 90 degrees
- moved R2 1.38 mm to (211.0, 105.6), turned to 0 degrees
- moved H2 1.10 mm to (169.6, 76.3)
- moved J5 0.66 mm to (217.5, 110.2)
- moved J4 0.50 mm to (212.7, 110.2)
- moved D4 0.40 mm to (248.6, 92.0)
- turned D2 to -90 degrees
- renumbered G*** to ?
Connections:
- H1 pad 1: (no net) -> GND
- H2 pad 1: (no net) -> GND
- H3 pad 1: (no net) -> GND
Routing:
- net LED split: track 481.3 -> 342.1 mm, vias 6 -> 4
- net +5Vlimited: track 474.0 -> 516.0 mm, vias 5 -> 0
- net IO37: track 45.4 -> 29.5 mm, vias 0 -> 1
- net +3V3: track 80.3 -> 76.2 mm, vias 1 -> 2
- net Net-(D3-Pad1): track 23.7 -> 20.2 mm
- net Net-(D7-Pad1): track 22.8 -> 20.4 mm
- net Net-(Q1-D): track 3.04 -> 5.28 mm
- net RST / IO15: track 29.0 -> 27.2 mm
- net Net-(D1-Pad1): track 21.8 -> 20.4 mm
- net SDA / IO8: track 17.9 -> 16.5 mm
- net Net-(J9-Pad2): track 42.9 -> 43.7 mm
- net GATE / IO45: track 14.6 -> 13.9 mm
- net IO38: track 26.3 -> 26.9 mm
- net IO42: track 16.3 -> 16.8 mm
- net GND: track 4.87 -> 4.59 mm, vias 54 -> 38

Commit message: submitted
Parts:
- added ?: LOGO, LOGO, F.Cu at (211.0, 90.6)
- moved ? 7.84 mm to (185.6, 95.4)
- moved J10 0.40 mm to (241.8, 141.9)
- moved J16 0.20 mm to (241.8, 102.3)
- moved LS1 0.20 mm to (191.0, 80.6)
- moved J15 0.16 mm to (241.8, 89.0)
Routing:
- net +5V: track 206.9 -> 206.2 mm
- net GND: vias 38 -> 39
- added copper zone on In1.Cu, net GND
- added copper zone on In2.Cu, net GND
Other:
- copper layers 2 -> 4
