File: PCB Shield.kicad_pcb (KiCad board)
At the start: 4 copper layers, 92 x 99 mm, 57 parts, among them J1 Conn_1to20, J10 TB002-500-02BE, J11 TB002-500-02BE, J12 TB002-500-02BE, J13 TB002-500-02BE, J14 TB002-500-02BE, J15 TB002-500-02BE, J16 TB002-500-02BE, J2 Conn_01x08_Socket, J3 Conn_1to20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

Commit message: last minute changes
Routing:
- net Net-(J14-Pad1): track 41.9 -> 40.0 mm
Changed lines of the file:
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@@
 		(capping no)
 		(filling no)
-		(zone_defaults)
 		(pcbplotparams
 			(layerselection 0x00000000_00000000_55555555_5755f5ff)
@@
 		(at 209.1705 126.3665 180)
 		(property "Reference" "R9"
-			(at 1 -0.5 180)
+			(at 1.9705 -0.6335 0)
 			(unlocked yes)
 			(layer "F.SilkS")
@@
 		(at 209.1705 122.3665 180)
 		(property "Reference" "R8"
-			(at 1 -0.5 180)
+			(at 1.9705 -0.8335 0)
 			(unlocked yes)
 			(layer "F.SilkS")
@@
 	)
 	(segment
-		(start 209.0485 126)
-		(end 210 126)
+		(start 209.4 125.2)
+		(end 209.3015 125.2985)
 		(width 0.2)
 		(layer "F.Cu")
@@
 	)
 	(segment
-		(start 208.347 125.2985)
-		(end 209.0485 126)
+		(start 209.3015 125.2985)
+		(end 208.347 125.2985)
 		(width 0.2)
 		(layer "F.Cu")
@@
 	)
 	(via
-		(at 210 126)
+		(at 209.4 125.2)
 		(size 0.6)
 		(drill 0.3)
@@
 	)
 	(segment
-		(start 210 126)
-		(end 210 155.8375)
+		(start 209.4 125.2)
+		(end 209.4 156.4375)
 		(width 0.2)
 		(layer "B.Cu")
@@
 	)
 	(segment
-		(start 210 155.8375)
+		(start 209.4 156.4375)
 		(end 208 157.8375)
 		(width 0.2)
@@
 		(net "DATA 3Y")
 	)
-	(segment
-		(start 209.2985 121.2985)
-		(end 210 122)
-		(width 0.2)
-		(layer "F.Cu")
-		(net "Net-(J14-Pad1)")
-	)
-	(segment
-		(start 208.347 121.2985)
-		(end 209.2985 121.2985)
-		(width 0.2)
-		(layer "F.Cu")
-		(net "Net-(J14-Pad1)")
-	)
 	(via
-		(at 210 122)
+		(at 208.347 121.2985)
 		(size 0.6)
 		(drill 0.3)
@@
 	)
 	(segment
-		(start 209 153.91875)
-		(end 205.08125 157.8375)
+		(start 208.4 121.3515)
+		(end 208.4 154.51875)
 		(width 0.2)
 		(layer "B.Cu")
@@
 	)
 	(segment
-		(start 209 126)
-		(end 209 153.91875)
-		(width 0.2)
-		(layer "B.Cu")
-		(net "Net-(J14-Pad1)")
-	)
-	(segment
-		(start 210 122)
-		(end 210 125)
+		(start 208.4 154.51875)
+		(end 205.08125 157.8375)
 		(width 0.2)
 		(layer "B.Cu")
@@
 	)
 	(segment
-		(start 210 125)
-		(end 209 126)
+		(start 205.08125 157.8375)
+		(end 203 157.8375)
 		(width 0.2)
 		(layer "B.Cu")
@@
 	)
 	(segment
-		(start 205.08125 157.8375)
-		(end 203 157.8375)
+		(start 208.347 121.2985)
+		(end 208.4 121.3515)
 		(width 0.2)
 		(layer "B.Cu")

Commit message: hopefully it pushes. Flipped the headers and shrunk down board
Parts:
- R1: value 10k -> 4k7
- R10: value 150 -> 220
- moved VR2 56.6 mm to (182.6, 102.8), turned to 180 degrees
- moved J3 52.0 mm to (182.2, 110.1), turned to 0 degrees
- moved J1 51.9 mm to (178.0, 110.2), turned to 0 degrees
- moved VR1 43.9 mm to (192.4, 110.6), turned to 180 degrees
- moved LS1 26.2 mm to (212.8, 95.2)
- moved ? 18.9 mm to (189.8, 77.0), turned to 180 degrees
- moved ? 16.4 mm to (202.4, 85.2)
- moved R5 15.7 mm to (187.5, 127.7), turned to 90 degrees
- moved J6 14.9 mm to (196.8, 129.4), turned to 0 degrees
- moved J7 14.8 mm to (193.0, 129.5), turned to 0 degrees
- moved R3 13.7 mm to (189.7, 129.1), turned to -90 degrees
- moved J2 12.8 mm to (175.8, 124.0)
- moved ? 12.1 mm to (202.8, 99.5), turned to -90 degrees
- moved H3 12.1 mm to (173.8, 150.4)
- moved D2 7.60 mm to (169.6, 139.0), turned to 180 degrees
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Connections:
- net SCL / IO9 renamed SCL / IO8
- net SDA / IO8 renamed SDA / IO7
- J6 pad 3: +5Vlimited -> +3V3
- J7 pad 3: +5Vlimited -> +3V3
- R3 pad 2: +5Vlimited -> +3V3
- R5 pad 2: +5Vlimited -> +3V3
Routing:
- net +5Vlimited: track 516.0 -> 339.7 mm
- net +3V3: track 76.2 -> 144.9 mm
- net EN1 / IO2: track 66.1 -> 18.9 mm, vias 1 -> 0
- net A1 / IO3: track 63.6 -> 18.8 mm, vias 1 -> 0
- net LED split: track 342.1 -> 298.4 mm
- net RST / IO15: track 27.2 -> 52.2 mm
- net PWM / IO16: track 48.5 -> 28.8 mm, vias 0 -> 1
- net IRQ / IO14: track 26.2 -> 43.3 mm
- net GND: track 4.59 -> 17.6 mm, vias 39 -> 35
- net MISO / Query: track 26.2 -> 33.8 mm
- net Net-(J9-Pad1): track 43.2 -> 49.8 mm
- net ADC1_3 / IO4: track 11.2 -> 17.7 mm, vias 0 -> 1
- net CS / IO10: track 26.5 -> 21.2 mm
- net SCLK: track 25.1 -> 30.0 mm
- net Net-(J4-Pin_8): track 4.59 -> 9.33 mm
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Other:
- board size 92 x 99 mm -> 84 x 99 mm
